Commit message: Update urdf

File: tang_description/urdf/tang.urdf (robot description, URDF)
Before this commit: robot tang, 1 links, 0 joints
Links:
- removed link map
- added link base_link; visual mesh filename=package://tang_description/base_link.obj scale=0.001 0.001 0.001
- added link left_wheel; visual mesh filename=package://tang_description/CuGoV3_Left.obj scale=0.001 0.001 0.001
- added link right_wheel; visual mesh filename=package://tang_description/CuGoV3_Right.obj scale=0.001 0.001 0.001
Joints:
- added joint left_wheel_joint: type continuous, parent base_link, child left_wheel, origin xyz=0 0.18 0 rpy=0.0 0.0 0.0, axis 0 0 1
- added joint right_wheel_joint: type continuous, parent base_link, child right_wheel, origin xyz=0 -0.18 0 rpy=0.0 0.0 0.0, axis 0 0 1
